File: makeTracer/circuit/maincircuit/maincircuit.kicad_sch (KiCad schematic)
At the start: 15 parts, among them IC1 PIC16F1778-I_SP, J1 PICKit3, J2 Sensor, J3 I^{2}C, SW1 SW_DPDT_x2, SW2 Reset, SW3 Red, SW4 Green

Commit message: wipp
Parts:
- removed IC1: PIC16F1778-I_SP, Package_DIP:DIP-28_W7.62mm_Socket_LongPads, symbol SamacSys:PIC16F1778-I_SP
- added IC1: PIC16F1778-I/SP, Package_DIP:DIP-28_W7.62mm_Socket_LongPads, symbol D4jikkenLibrary:PIC16F1778-I/SP
Connections:
- net 16x2LEDs/Clock: now also IC1.23 (RB2)
- net 16x2LEDs/Data: now also IC1.22 (RB1)
- net 16x2LEDs/Flash: now also IC1.24 (RB3)
- net GND: now also IC1.19 (VSS_2), IC1.8 (VSS_1)
- net I^{2}C_SCL: now also IC1.18 (RC7)
- net I^{2}C_SDA: now also IC1.21 (RB0)
- net Motordrive/L_PWM: now also IC1.12 (RC1)
- net Motordrive/L_SEL1: now also IC1.13 (RC2)
- net Motordrive/L_SEL2: now also IC1.14 (RC3)
- net Motordrive/R_PWM: now also IC1.17 (RC6)
- net Motordrive/R_SEL1: now also IC1.16 (RC5)
- net Motordrive/R_SEL2: now also IC1.15 (RC4)
- net PICKit3_ICSPCLK: now also IC1.27 (RB6/ICSPCLK)
- net PICKit3_ICSPDAT: now also IC1.28 (RB7/ICSPDAT)
- net PICKit3_MCLR: now also IC1.1 (VPP/~{MCLR}/RE3)
- net Sensor_AN: now also IC1.3 (RA1)
- net Sensor_DI: now also IC1.2 (RA0)
- net Sensor_SEL1: now also IC1.4 (RA2)
- net Sensor_SEL2: now also IC1.5 (RA3)
- net VDD: now also IC1.20 (VDD)
- net at LS1.1: now also IC1.9 (RA7)
- net at SW4.2: now also IC1.7 (RA5)
- net at SW3.2: now also IC1.6 (RA4)

Commit message: done: maincircuit
Parts:
- PWR1: renamed from D1; value LED_Dual_AKA -> PowerIndicator
- R1: footprint Resistor_THT:R_Axial_DIN0207_L6.3mm_D2.5mm_P10.16mm_Horizontal -> Resistor_THT:R_Axial_DIN0207_L6.3mm_D2.5mm_P2.54mm_Vertical
Connections:
- net 16x2LEDs/Select_Red: now reaches IC1.25 (RB4)
- net 16x2LEDs/Select_Green: now reaches IC1.26 (RB5)
Other:
- sheet 16x2LEDs ports: added Select_Green, Select_Red; removed none

Commit message: fix: yabai jumper
Parts:
- BT1: footprint Connector_PinHeader_2.54mm:PinHeader_1x02_P2.54mm_Horizontal -> Connector_PinHeader_2.54mm:PinHeader_1x02_P2.54mm_Vertical
- R2: footprint Resistor_THT:R_Axial_DIN0207_L6.3mm_D2.5mm_P2.54mm_Vertical -> Resistor_THT:R_Axial_DIN0207_L6.3mm_D2.5mm_P5.08mm_Vertical
Changed lines of the file:
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@@
       (effects (font (size 1.27 1.27)) (justify left))
     )
-    (property "Footprint" "Resistor_THT:R_Axial_DIN0207_L6.3mm_D2.5mm_P2.54mm_Vertical" (at 207.772 113.03 90)
+    (property "Footprint" "Resistor_THT:R_Axial_DIN0207_L6.3mm_D2.5mm_P5.08mm_Vertical" (at 207.772 113.03 90)
       (effects (font (size 1.27 1.27)) hide)
     )
@@
       (effects (font (size 1.27 1.27)) (justify left))
     )
-    (property "Footprint" "Connector_PinHeader_2.54mm:PinHeader_1x02_P2.54mm_Horizontal" (at 254 115.951 90)
+    (property "Footprint" "Connector_PinHeader_2.54mm:PinHeader_1x02_P2.54mm_Vertical" (at 254 115.951 90)
       (effects (font (size 1.27 1.27)) hide)
     )
