File: makeTracer/circuit/maincircuit/16x2LEDs.kicad_sch (KiCad schematic)
At the start: 2 parts, among them U2 74HC595, U3 74HC595

Commit message: wippu
Parts:
- added P1, P2: AirWirePort, Connector_PinHeader_2.54mm:PinHeader_1x08_P2.54mm_Vertical, symbol Connector_Generic:Conn_01x08
Connections:
- net LED1: now also P1.1 (Pin_1)
- net LED10: now also P2.2 (Pin_2)
- net LED11: now also P2.3 (Pin_3)
- net LED12: now also P2.4 (Pin_4)
- net LED13: now also P2.5 (Pin_5)
- net LED14: now also P2.6 (Pin_6)
- net LED15: now also P2.7 (Pin_7)
- net LED16: now also P2.8 (Pin_8)
- net LED2: now also P1.2 (Pin_2)
- net LED3: now also P1.3 (Pin_3)
- net LED4: now also P1.4 (Pin_4)
- net LED5: now also P1.5 (Pin_5)
- net LED6: now also P1.6 (Pin_6)
- net LED7: now also P1.7 (Pin_7)
- net LED8: now also P1.8 (Pin_8)
- net LED9: now also P2.1 (Pin_1)
Changed lines of the file:
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@@
+    (stroke (width 0) (type default))
+  )
+  (wire (pts (xy 62.23 101.6) (xy 72.39 101.6))
     (stroke (width 0) (type default))
   )
@@
     (stroke (width 0) (type default))
   )
+  (wire (pts (xy 113.03 99.06) (xy 123.19 99.06))
+    (stroke (width 0) (type default))
+  )
   (bus (pts (xy 59.69 52.07) (xy 59.69 54.61))
     (stroke (width 0) (type default))
@@
     (stroke (width 0) (type default))
   )
+  (wire (pts (xy 113.03 114.3) (xy 123.19 114.3))
+    (stroke (width 0) (type default))
+  )
   (wire (pts (xy 49.53 46.99) (xy 57.15 46.99))
     (stroke (width 0) (type default))
@@
     (stroke (width 0) (type default))
   )
+  (wire (pts (xy 113.03 104.14) (xy 123.19 104.14))
+    (stroke (width 0) (type default))
+  )
   (bus (pts (xy 59.69 54.61) (xy 59.69 96.52))
     (stroke (width 0) (type default))
@@
     (stroke (width 0) (type default))
   )
+  (wire (pts (xy 113.03 111.76) (xy 123.19 111.76))
+    (stroke (width 0) (type default))
+  )
+  (wire (pts (xy 62.23 106.68) (xy 72.39 106.68))
+    (stroke (width 0) (type default))
+  )
   (bus (pts (xy 110.49 41.91) (xy 110.49 44.45))
     (stroke (width 0) (type default))
@@
     (stroke (width 0) (type default))
   )
+  (wire (pts (xy 62.23 114.3) (xy 72.39 114.3))
+    (stroke (width 0) (type default))
+  )
   (wire (pts (xy 100.33 44.45) (xy 107.95 44.45))
     (stroke (width 0) (type default))
@@
     (stroke (width 0) (type default))
   )
+  (wire (pts (xy 113.03 116.84) (xy 123.19 116.84))
+    (stroke (width 0) (type default))
+  )
   (bus (pts (xy 59.69 106.68) (xy 59.69 109.22))
     (stroke (width 0) (type default))
@@
     (stroke (width 0) (type default))
   )
+  (wire (pts (xy 62.23 109.22) (xy 72.39 109.22))
+    (stroke (width 0) (type default))
+  )
+  (wire (pts (xy 113.03 101.6) (xy 123.19 101.6))
+    (stroke (width 0) (type default))
+  )
+  (wire (pts (xy 62.23 116.84) (xy 72.39 116.84))
+    (stroke (width 0) (type default))
+  )
   (bus (pts (xy 59.69 109.22) (xy 59.69 111.76))
     (stroke (width 0) (type default))
@@
     (stroke (width 0) (type default))
   )
+  (wire (pts (xy 62.23 99.06) (xy 72.39 99.06))
+    (stroke (width 0) (type default))
+  )
+  (wire (pts (xy 62.23 111.76) (xy 72.39 111.76))
+    (stroke (width 0) (type default))
+  )
   (bus (pts (xy 59.69 49.53) (xy 59.69 52.07))
     (stroke (width 0) (type default))
@@
     (stroke (width 0) (type default))
   )
+  (wire (pts (xy 62.23 104.14) (xy 72.39 104.14))
+    (stroke (width 0) (type default))
+  )
+  (wire (pts (xy 113.03 106.68) (xy 123.19 106.68))
+    (stroke (width 0) (type default))
+  )
   (wire (pts (xy 65.405 57.15) (xy 65.405 34.29))
     (stroke (width 0) (type default))
   )
+  (wire (pts (xy 113.03 109.22) (xy 123.19 109.22))
+    (stroke (width 0) (type default))
+  )
   (bus (pts (xy 110.49 39.37) (xy 110.49 41.91))
     (stroke (width 0) (type default))
@@
     (effects (font (size 1.27 1.27)) (justify left bottom))
   )
+  (label "LED15" (at 116.84 114.3 0) (fields_autoplaced)
+    (effects (font (size 1.27 1.27)) (justify left bottom))
+  )
+  (label "LED7" (at 64.77 114.3 0) (fields_autoplaced)
+    (effects (font (size 1.27 1.27)) (justify left bottom))
+  )
   (label "LED3" (at 50.8 39.37 0) (fields_autoplaced)
     (effects (font (size 1.27 1.27)) (justify left bottom))
@@
     (effects (font (size 1.27 1.27)) (justify left bottom))
   )
+  (label "LED1" (at 64.77 99.06 0) (fields_autoplaced)
+    (effects (font (size 1.27 1.27)) (justify left bottom))
+  )
+  (label "LED5" (at 64.77 109.22 0) (fields_autoplaced)
+    (effects (font (size 1.27 1.27)) (justify left bottom))
+  )
+  (label "LED11" (at 116.84 104.14 0) (fields_autoplaced)
+    (effects (font (size 1.27 1.27)) (justify left bottom))
+  )
+  (label "LED16" (at 116.84 116.84 0) (fields_autoplaced)
+    (effects (font (size 1.27 1.27)) (justify left bottom))
+  )
   (label "LED8" (at 50.8 52.07 0) (fields_autoplaced)
     (effects (font (size 1.27 1.27)) (justify left bottom))
   )
+  (label "LED12" (at 116.84 106.68 0) (fields_autoplaced)
+    (effects (font (size 1.27 1.27)) (justify left bottom))
+  )
+  (label "LED2" (at 64.77 101.6 0) (fields_autoplaced)
+    (effects (font (size 1.27 1.27)) (justify left bottom))
+  )
   (label "LED1" (at 50.8 34.29 0) (fields_autoplaced)
     (effects (font (size 1.27 1.27)) (justify left bottom))
@@
     (effects (font (size 1.27 1.27)) (justify left bottom))
   )
+  (label "LED4" (at 64.77 106.68 0) (fields_autoplaced)
+    (effects (font (size 1.27 1.27)) (justify left bottom))
+  )
   (label "LED5" (at 50.8 44.45 0) (fields_autoplaced)
     (effects (font (size 1.27 1.27)) (justify left bottom))
@@
     (effects (font (size 1.27 1.27)) (justify left bottom))
   )
+  (label "LED9" (at 116.84 99.06 0) (fields_autoplaced)
+    (effects (font (size 1.27 1.27)) (justify left bottom))
+  )
+  (label "LED6" (at 64.77 111.76 0) (fields_autoplaced)
+    (effects (font (size 1.27 1.27)) (justify left bottom))
+  )
   (label "LED7" (at 50.8 49.53 0) (fields_autoplaced)
     (effects (font (size 1.27 1.27)) (justify left bottom))
   )
+  (label "LED8" (at 64.77 116.84 0) (fields_autoplaced)
+    (effects (font (size 1.27 1.27)) (justify left bottom))
+  )
+  (label "LED10" (at 116.84 101.6 0) (fields_autoplaced)
+    (effects (font (size 1.27 1.27)) (justify left bottom))
+  )
   (label "LED14" (at 101.6 46.99 0) (fields_autoplaced)
     (effects (font (size 1.27 1.27)) (justify left bottom))
@@
     (effects (font (size 1.27 1.27)) (justify left bottom))
   )
+  (label "LED3" (at 64.77 104.14 0) (fields_autoplaced)
+    (effects (font (size 1.27 1.27)) (justify left bottom))
+  )
+  (label "LED14" (at 116.84 111.76 0) (fields_autoplaced)
+    (effects (font (size 1.27 1.27)) (justify left bottom))
+  )
+  (label "LED13" (at 116.84 109.22 0) (fields_autoplaced)
+    (effects (font (size 1.27 1.27)) (justify left bottom))
+  )
   (label "LED9" (at 101.6 34.29 0) (fields_autoplaced)
     (effects (font (size 1.27 1.27)) (justify left bottom))
@@
   (hierarchical_label "~{Clear}" (shape input) (at 29.21 41.91 180) (fields_autoplaced)
     (effects (font (size 1.27 1.27)) (justify right))
+  )
+  (symbol (lib_id "Connector_Generic:Conn_01x08") (at 77.47 106.68 0) (unit 1)
+    (in_bom yes) (on_board yes) (dnp no) (fields_autoplaced)
+    (property "Reference" "P1" (at 80.01 106.68 0)
+      (effects (font (size 1.27 1.27)) (justify left))
+    )
+    (property "Value" "AirWirePort" (at 80.01 109.22 0)
+      (effects (font (size 1.27 1.27)) (justify left))
+    )
+    (property "Footprint" "Connector_PinHeader_2.54mm:PinHeader_1x08_P2.54mm_Vertical" (at 77.47 106.68 0)
+      (effects (font (size 1.27 1.27)) hide)
+    )
+    (property "Datasheet" "~" (at 77.47 106.68 0)
+      (effects (font (size 1.27 1.27)) hide)
+    )
+    (pin "1")
+    (pin "2")
+    (pin "3")
+    (pin "4")
+    (pin "5")
+    (pin "6")
+    (pin "7")
+    (pin "8")
+    (instances
+      (project "maincircuit"
+        (path "/a588b4f4-c52b-4b14-933c-cea644bb9512/db89b617-3486-457b-86f5-38eff07d4cbf"
+          (reference "P1") (unit 1)
+        )
+      )
+    )
   )
   (symbol (lib_id "74xx:74HC595") (at 90.17 44.45 0) (unit 1)
@@
         )
       )
+    )
+  )
+  (symbol (lib_id "Connector_Generic:Conn_01x08") (at 128.27 106.68 0) (unit 1)
+    (in_bom yes) (on_board yes) (dnp no) (fields_autoplaced)
+    (property "Reference" "P2" (at 130.81 106.68 0)
+      (effects (font (size 1.27 1.27)) (justify left))
+    )
+    (property "Value" "AirWirePort" (at 130.81 109.22 0)
+      (effects (font (size 1.27 1.27)) (justify left))
+    )
+    (property "Footprint" "Connector_PinHeader_2.54mm:PinHeader_1x08_P2.54mm_Vertical" (at 128.27 106.68 0)
+      (effects (font (size 1.27 1.27)) hide)
+    )
+    (property "Datasheet" "~" (at 128.27 106.68 0)
+      (effects (font (size 1.27 1.27)) hide)
+    )
+    (pin "1")
+    (pin "2")
+    (pin "3")
+    (pin "4")
+    (pin "5")
+    (pin "6")
+    (pin "7")
+    (pin "8")
+    (instances
+      (project "maincircuit"
+        (path "/a588b4f4-c52b-4b14-933c-cea644bb9512/db89b617-3486-457b-86f5-38eff07d4cbf"
+          (reference "P2") (unit 1)
+        )
+      )

Commit message: done: maincircuit
Parts:
- removed P1, P2: AirWirePort, Connector_PinHeader_2.54mm:PinHeader_1x08_P2.54mm_Vertical, symbol Connector_Generic:Conn_01x08
- added C1 (x2): 0.1u_pass, Capacitor_THT:C_Disc_D5.0mm_W2.5mm_P2.50mm, symbol Device:C
- added LED1, LED10, LED11, LED12, LED13, LED14, LED15, LED16, LED2, LED3, LED4, LED5, LED6, LED7, LED8, LED9: Circle, LED_THT:LED_D3.0mm-3, symbol Device:LED_Dual_AKA
- added P1: FrontsidePort, Connector_PinHeader_2.54mm:PinHeader_1x02_P2.54mm_Vertical, symbol Connector_Generic:Conn_01x02
- added R11, R13, R14, R15, R16, R17, R18, R19, R20, R21, R22, R23, R24, R25, R26: 470, Resistor_THT:R_Axial_DIN0207_L6.3mm_D2.5mm_P2.54mm_Vertical, symbol Device:R
- added R12: 470, Resistor_THT:R_Axial_DIN0207_L6.3mm_D2.5mm_P15.24mm_Horizontal, symbol Device:R
- added Tr1, Tr2: DTC114E, Package_TO_SOT_THT:TO-92, symbol Transistor_BJT:DTC114E
Connections:
- net GND: now also C1.2, C1.2
- net LED1: now also R11.2
- net LED10: now also R20.2
- net LED11: now also R21.2
- net LED12: now also R22.2
- net LED13: now also R23.2
- net LED14: now also R24.2
- net LED15: now also R25.2
- net LED16: now also R26.2
- net LED2: now also R12.2
- net LED3: now also R13.2
- net LED4: now also R14.2
- net LED5: now also R15.2
- net LED6: now also R16.2
- net LED7: now also R17.2
- net LED8: now also R18.2
- net LED9: now also R19.2
- net VDD: now also C1.1, C1.1, Tr1.3 (C), Tr2.3 (C)
- new net: LED4.2 (K), R14.1
- new net: LED12.2 (K), R22.1
- new net: LED1.2 (K), R11.1
- new net: LED3.2 (K), R13.1
- new net: LED11.2 (K), R21.1
- new net: LED13.2 (K), R23.1
- new net: LED9.2 (K), R19.1
- new net: LED15.2 (K), R25.1
- new net: LED14.2 (K), R24.1
- new net: LED16.2 (K), R26.1
- new net: LED10.2 (K), R20.1
- new net: LED5.2 (K), R15.1
- new net: LED8.2 (K), R18.1
- new net: LED6.2 (K), R16.1
- new net: LED7.2 (K), R17.1
- new net: LED2.2 (K), R12.1
- new net Green_Src: LED1.3 (A2), LED10.3 (A2), LED11.3 (A2), LED12.3 (A2), LED13.3 (A2), LED14.3 (A2), LED15.3 (A2), LED16.3 (A2), LED2.3 (A2), LED3.3 (A2), LED4.3 (A2), LED5.3 (A2), LED6.3 (A2), LED7.3 (A2), LED8.3 (A2), LED9.3 (A2), P1.2 (Pin_2), Tr2.2 (E)
- new net Red_Src: LED1.1 (A1), LED10.1 (A1), LED11.1 (A1), LED12.1 (A1), LED13.1 (A1), LED14.1 (A1), LED15.1 (A1), LED16.1 (A1), LED2.1 (A1), LED3.1 (A1), LED4.1 (A1), LED5.1 (A1), LED6.1 (A1), LED7.1 (A1), LED8.1 (A1), LED9.1 (A1), P1.1 (Pin_1), Tr1.2 (E)
- new net Select_Green: Tr2.1 (B)
- new net Select_Red: Tr1.1 (B)
Other:
- moved on the sheet: U2, U3

Commit message: fix: yabai jumper
Parts:
- R11, R13, R14, R15, R16, R17, R18, R19, R20, R21, R22, R23, R24, R25, R26: footprint Resistor_THT:R_Axial_DIN0207_L6.3mm_D2.5mm_P2.54mm_Vertical -> Resistor_THT:R_Axial_DIN0207_L6.3mm_D2.5mm_P7.62mm_Horizontal
- R12: footprint Resistor_THT:R_Axial_DIN0207_L6.3mm_D2.5mm_P15.24mm_Horizontal -> Resistor_THT:R_Axial_DIN0207_L6.3mm_D2.5mm_P7.62mm_Horizontal
Changed lines of the file:
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@@
   (junction (at 215.9 45.72) (diameter 0) (color 0 0 0 0)
   )
-  (junction (at 228.6 147.574) (diameter 0) (color 0 0 0 0)
-  )
   (junction (at 114.3 50.8) (diameter 0) (color 0 0 0 0)
   )
@@
   )
   (junction (at 165.1 45.72) (diameter 0) (color 0 0 0 0)
-  )
-  (junction (at 228.6 132.334) (diameter 0) (color 0 0 0 0)
   )
   (junction (at 226.06 45.72) (diameter 0) (color 0 0 0 0)
@@
     (stroke (width 0) (type default))
   )
-  (wire (pts (xy 246.38 143.764) (xy 246.38 147.574))
+  (wire (pts (xy 246.38 143.764) (xy 246.38 149.86))
     (stroke (width 0) (type default))
   )
@@
     (stroke (width 0) (type default))
   )
-  (wire (pts (xy 228.6 129.54) (xy 228.6 132.334))
+  (wire (pts (xy 228.6 129.54) (xy 228.6 135.89))
     (stroke (width 0) (type default))
   )
@@
     (stroke (width 0) (type default))
   )
-  (wire (pts (xy 228.6 132.334) (xy 228.6 135.89))
-    (stroke (width 0) (type default))
-  )
-  (wire (pts (xy 228.6 143.51) (xy 228.6 147.574))
+  (wire (pts (xy 228.6 143.51) (xy 228.6 149.86))
     (stroke (width 0) (type default))
   )
@@
     (stroke (width 0) (type default))
   )
-  (wire (pts (xy 228.6 132.334) (xy 246.38 132.334))
-    (stroke (width 0) (type default))
-  )
   (wire (pts (xy 170.18 50.8) (xy 160.02 50.8))
     (stroke (width 0) (type default))
@@
     (stroke (width 0) (type default))
   )
-  (wire (pts (xy 246.38 132.334) (xy 246.38 136.144))
+  (wire (pts (xy 246.38 129.54) (xy 246.38 136.144))
     (stroke (width 0) (type default))
   )
@@
     (stroke (width 0) (type default))
   )
-  (wire (pts (xy 228.6 147.574) (xy 246.38 147.574))
-    (stroke (width 0) (type default))
-  )
   (wire (pts (xy 139.7 45.72) (xy 149.86 45.72))
     (stroke (width 0) (type default))
@@
   )
   (wire (pts (xy 139.7 58.42) (xy 139.7 45.72))
-    (stroke (width 0) (type default))
-  )
-  (wire (pts (xy 228.6 147.574) (xy 228.6 149.86))
     (stroke (width 0) (type default))
   )
@@
       (effects (font (size 1.27 1.27)) (justify left))
     )
-    (property "Footprint" "Resistor_THT:R_Axial_DIN0207_L6.3mm_D2.5mm_P2.54mm_Vertical" (at 74.422 101.6 90)
+    (property "Footprint" "Resistor_THT:R_Axial_DIN0207_L6.3mm_D2.5mm_P7.62mm_Horizontal" (at 74.422 101.6 90)
       (effects (font (size 1.27 1.27)) hide)
     )
@@
       (effects (font (size 1.27 1.27)) (justify left))
     )
-    (property "Footprint" "Resistor_THT:R_Axial_DIN0207_L6.3mm_D2.5mm_P2.54mm_Vertical" (at 191.262 101.6 90)
+    (property "Footprint" "Resistor_THT:R_Axial_DIN0207_L6.3mm_D2.5mm_P7.62mm_Horizontal" (at 191.262 101.6 90)
       (effects (font (size 1.27 1.27)) hide)
     )
@@
       (effects (font (size 1.27 1.27)) (justify left))
     )
-    (property "Footprint" "Resistor_THT:R_Axial_DIN0207_L6.3mm_D2.5mm_P2.54mm_Vertical" (at 160.782 101.6 90)
+    (property "Footprint" "Resistor_THT:R_Axial_DIN0207_L6.3mm_D2.5mm_P7.62mm_Horizontal" (at 160.782 101.6 90)
       (effects (font (size 1.27 1.27)) hide)
     )
@@
       (effects (font (size 1.27 1.27)) (justify left))
     )
-    (property "Footprint" "Resistor_THT:R_Axial_DIN0207_L6.3mm_D2.5mm_P2.54mm_Vertical" (at 231.902 101.6 90)
+    (property "Footprint" "Resistor_THT:R_Axial_DIN0207_L6.3mm_D2.5mm_P7.62mm_Horizontal" (at 231.902 101.6 90)
       (effects (font (size 1.27 1.27)) hide)
     )
@@
       (effects (font (size 1.27 1.27)) (justify left))
     )
-    (property "Footprint" "Resistor_THT:R_Axial_DIN0207_L6.3mm_D2.5mm_P2.54mm_Vertical" (at 94.742 101.6 90)
+    (property "Footprint" "Resistor_THT:R_Axial_DIN0207_L6.3mm_D2.5mm_P7.62mm_Horizontal" (at 94.742 101.6 90)
       (effects (font (size 1.27 1.27)) hide)
     )
@@
       (effects (font (size 1.27 1.27)) (justify left))
     )
-    (property "Footprint" "Resistor_THT:R_Axial_DIN0207_L6.3mm_D2.5mm_P2.54mm_Vertical" (at 201.422 101.6 90)
+    (property "Footprint" "Resistor_THT:R_Axial_DIN0207_L6.3mm_D2.5mm_P7.62mm_Horizontal" (at 201.422 101.6 90)
       (effects (font (size 1.27 1.27)) hide)
     )
@@
       (effects (font (size 1.27 1.27)) (justify left))
     )
-    (property "Footprint" "Resistor_THT:R_Axial_DIN0207_L6.3mm_D2.5mm_P2.54mm_Vertical" (at 170.942 101.6 90)
+    (property "Footprint" "Resistor_THT:R_Axial_DIN0207_L6.3mm_D2.5mm_P7.62mm_Horizontal" (at 170.942 101.6 90)
       (effects (font (size 1.27 1.27)) hide)
     )
@@
       (effects (font (size 1.27 1.27)) (justify left))
     )
-    (property "Footprint" "Resistor_THT:R_Axial_DIN0207_L6.3mm_D2.5mm_P2.54mm_Vertical" (at 145.542 101.6 90)
+    (property "Footprint" "Resistor_THT:R_Axial_DIN0207_L6.3mm_D2.5mm_P7.62mm_Horizontal" (at 145.542 101.6 90)
       (effects (font (size 1.27 1.27)) hide)
     )
@@
       (effects (font (size 1.27 1.27)) (justify left))
     )
-    (property "Footprint" "Resistor_THT:R_Axial_DIN0207_L6.3mm_D2.5mm_P2.54mm_Vertical" (at 115.062 101.6 90)
+    (property "Footprint" "Resistor_THT:R_Axial_DIN0207_L6.3mm_D2.5mm_P7.62mm_Horizontal" (at 115.062 101.6 90)
       (effects (font (size 1.27 1.27)) hide)
     )
@@
       (effects (font (size 1.27 1.27)) (justify left))
     )
-    (property "Footprint" "Resistor_THT:R_Axial_DIN0207_L6.3mm_D2.5mm_P2.54mm_Vertical" (at 181.102 101.6 90)
+    (property "Footprint" "Resistor_THT:R_Axial_DIN0207_L6.3mm_D2.5mm_P7.62mm_Horizontal" (at 181.102 101.6 90)
       (effects (font (size 1.27 1.27)) hide)
     )
@@
     )
   )
+  (symbol (lib_id "power:GND") (at 246.38 149.86 0) (unit 1)
+    (in_bom yes) (on_board yes) (dnp no) (fields_autoplaced)
+    (property "Reference" "#PWR035" (at 246.38 156.21 0)
+      (effects (font (size 1.27 1.27)) hide)
+    )
+    (property "Value" "GND" (at 246.38 154.94 0)
+      (effects (font (size 1.27 1.27)))
+    )
+    (property "Footprint" "" (at 246.38 149.86 0)
+      (effects (font (size 1.27 1.27)) hide)
+    )
+    (property "Datasheet" "" (at 246.38 149.86 0)
+      (effects (font (size 1.27 1.27)) hide)
+    )
+    (pin "1")
+    (instances
+      (project "maincircuit"
+        (path "/a588b4f4-c52b-4b14-933c-cea644bb9512/db89b617-3486-457b-86f5-38eff07d4cbf"
+          (reference "#PWR035") (unit 1)
+        )
+      )
+    )
+  )
   (symbol (lib_id "Device:LED_Dual_AKA") (at 172.72 83.82 90) (unit 1)
     (in_bom yes) (on_board yes) (dnp no)
@@
       (effects (font (size 1.27 1.27)) (justify left))
     )
-    (property "Footprint" "Resistor_THT:R_Axial_DIN0207_L6.3mm_D2.5mm_P2.54mm_Vertical" (at 104.902 101.6 90)
+    (property "Footprint" "Resistor_THT:R_Axial_DIN0207_L6.3mm_D2.5mm_P7.62mm_Horizontal" (at 104.902 101.6 90)
       (effects (font (size 1.27 1.27)) hide)
     )
@@
     )
   )
+  (symbol (lib_id "power:VDD") (at 246.38 129.54 0) (unit 1)
+    (in_bom yes) (on_board yes) (dnp no) (fields_autoplaced)
+    (property "Reference" "#PWR032" (at 246.38 133.35 0)
+      (effects (font (size 1.27 1.27)) hide)
+    )
+    (property "Value" "VDD" (at 246.38 124.46 0)
+      (effects (font (size 1.27 1.27)))
+    )
+    (property "Footprint" "" (at 246.38 129.54 0)
+      (effects (font (size 1.27 1.27)) hide)
+    )
+    (property "Datasheet" "" (at 246.38 129.54 0)
+      (effects (font (size 1.27 1.27)) hide)
+    )
+    (pin "1")
+    (instances
+      (project "maincircuit"
+        (path "/a588b4f4-c52b-4b14-933c-cea644bb9512/db89b617-3486-457b-86f5-38eff07d4cbf"
+          (reference "#PWR032") (unit 1)
+        )
+      )
+    )
+  )
   (symbol (lib_id "Device:R") (at 127 101.6 0) (unit 1)
     (in_bom yes) (on_board yes) (dnp no)
@@
       (effects (font (size 1.27 1.27)) (justify left))
     )
-    (property "Footprint" "Resistor_THT:R_Axial_DIN0207_L6.3mm_D2.5mm_P2.54mm_Vertical" (at 125.222 101.6 90)
+    (property "Footprint" "Resistor_THT:R_Axial_DIN0207_L6.3mm_D2.5mm_P7.62mm_Horizontal" (at 125.222 101.6 90)
       (effects (font (size 1.27 1.27)) hide)
     )
@@
       (effects (font (size 1.27 1.27)) (justify left))
     )
-    (property "Footprint" "Resistor_THT:R_Axial_DIN0207_L6.3mm_D2.5mm_P15.24mm_Horizontal" (at 84.582 101.6 90)
+    (property "Footprint" "Resistor_THT:R_Axial_DIN0207_L6.3mm_D2.5mm_P7.62mm_Horizontal" (at 84.582 101.6 90)
       (effects (font (size 1.27 1.27)) hide)
     )
@@
       (effects (font (size 1.27 1.27)) (justify left))
     )
-    (property "Footprint" "Resistor_THT:R_Axial_DIN0207_L6.3mm_D2.5mm_P2.54mm_Vertical" (at 135.382 101.6 90)
+    (property "Footprint" "Resistor_THT:R_Axial_DIN0207_L6.3mm_D2.5mm_P7.62mm_Horizontal" (at 135.382 101.6 90)
       (effects (font (size 1.27 1.27)) hide)
     )
@@
       (effects (font (size 1.27 1.27)) (justify left))
     )
-    (property "Footprint" "Resistor_THT:R_Axial_DIN0207_L6.3mm_D2.5mm_P2.54mm_Vertical" (at 211.582 101.6 90)
+    (property "Footprint" "Resistor_THT:R_Axial_DIN0207_L6.3mm_D2.5mm_P7.62mm_Horizontal" (at 211.582 101.6 90)
       (effects (font (size 1.27 1.27)) hide)
     )
@@
       (effects (font (size 1.27 1.27)) (justify left))
     )
-    (property "Footprint" "Resistor_THT:R_Axial_DIN0207_L6.3mm_D2.5mm_P2.54mm_Vertical" (at 221.742 101.6 90)
-      (effects (font (size 1.27 1.27)) hide)
-    )
+    (property "Footprint" "Resistor_THT:R_Axial_DIN0207_L6.3mm_D2.5mm_P7.62mm_Horizontal" (at 221.742 101.6 90)
+      (effects (font (size 1.27 1.27)) hide)
+    )
