File: firstTracer/ciruit/ciruit.kicad_sch (KiCad schematic)
At the start: 21 parts, among them IC1 PIC16F1778-I_SP, J1 PicKit3, SW1 Reset, SW2 Start

Commit message: jikken2: fix circuit
Parts:
- LS1: footprint (none) -> Buzzer_Beeper:Buzzer_12x9.5RM7.6
Connections:
- net LSensor renamed sensor/SensorL
- net PWM_MotorL renamed motor/PWM_MotorL
- net PWM_MotorR renamed motor/SEL2_MotorR
- net RSensor renamed sensor/SensorR
- net SEL1_MotorL renamed motor/SEL2_MotorL
- net SEL1_MotorR renamed motor/SEL1_MotorR
- net SEL2_MotorL renamed motor/SEL1_MotorL
- net SEL2_MotorR renamed motor/PWM_MotorR
Other:
- sheet motor ports: added PWM_MotorL, PWM_MotorR, SEL1_MotorL, SEL1_MotorR, SEL2_MotorL, SEL2_MotorR; removed none
- sheet sensor ports: added SensorL, SensorR; removed none
- note removed: "6/18 2023"
- note removed: "MainCircuit"
- company: (none) -> KCCTD4-8
- title: (none) -> LineTracer-Practice

Commit message: complete: circuit
Parts:
- R9: value 10kΩ -> 10kR
Changed lines of the file:
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@@
     (company "KCCTD4-8")
     (comment 1 "*Unless otherwise noted, resistors used are 1/4W resistors.")
-    (comment 2 ">>>UNCHECKED CIRCUIT<<<")
   )
   (junction (at 208.915 128.27) (diameter 0) (color 0 0 0 0)
@@
       (effects (font (size 1.27 1.27)) (justify left))
     )
-    (property "Value" "10kΩ" (at 85.09 41.275 0)
-      (effects (font (size 1.27 1.27)) (justify left))
-    )
+    (property "Value" "10kR" (at 85.09 41.275 0)
+      (effects (font (size 1.27 1.27)) (justify left))
+    )
