File: firstTracer/ciruit/motor.kicad_sch (KiCad schematic)
At the start: 16 parts, among them M1 Motor_DC_Left, M2 Motor_DC_Right, Q1 MP4212_Q_, Q2 MP4212_Q_, U1 TC74HC00AP

Commit message: jikken2: fix circuit
Other:
- note removed: "6/18 2023"
- note removed: "MotorUnit"
- company: (none) -> KCCTD4-8
- title: (none) -> LineTracer-Practice-MotorDrive
Changed lines of the file:
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@@
 (kicad_sch (version 20230121) (generator eeschema)
   (paper "A4")
+  (title_block
+    (title "LineTracer-Practice-MotorDrive")
+    (date "2023-06-18")
+    (rev "ALPHA")
+    (company "KCCTD4-8")
+    (comment 1 "*Unless otherwise noted, resistors used are 1/4W resistors.")
+    (comment 2 ">>>UNCHECKED CIRCUIT<<<")
+  )
   (junction (at 101.6 139.7) (diameter 0) (color 0 0 0 0)
   )
@@
     (stroke (width 0) (type default))
   )
-  (text "MotorUnit" (at 187.325 191.135 0)
-    (effects (font (size 2.54 2.54) (thickness 0.508) bold italic) (justify left bottom))
-  )
-  (text "6/18 2023" (at 207.645 194.31 0)
-    (effects (font (size 1.27 1.27) bold) (justify left bottom))
-  )
-  (global_label "PWM_MotorL" (shape input) (at 37.465 66.675 180) (fields_autoplaced)
-    (effects (font (size 1.27 1.27)) (justify right))
-    (property "Intersheetrefs" "${INTERSHEET_REFS}" (at 23.1294 66.675 0)
-      (effects (font (size 1.27 1.27)) (justify right) hide)
-    )
-  )
-  (global_label "SEL2_MotorL" (shape input) (at 37.465 74.93 180) (fields_autoplaced)
-    (effects (font (size 1.27 1.27)) (justify right))
-    (property "Intersheetrefs" "${INTERSHEET_REFS}" (at 22.7061 74.93 0)
-      (effects (font (size 1.27 1.27)) (justify right) hide)
-    )
-  )
-  (global_label "PWM_MotorR" (shape input) (at 170.815 66.675 180) (fields_autoplaced)
-    (effects (font (size 1.27 1.27)) (justify right))
-    (property "Intersheetrefs" "${INTERSHEET_REFS}" (at 156.2375 66.675 0)
-      (effects (font (size 1.27 1.27)) (justify right) hide)
-    )
-  )
-  (global_label "SEL1_MotorL" (shape input) (at 37.465 58.42 180) (fields_autoplaced)
-    (effects (font (size 1.27 1.27)) (justify right))
-    (property "Intersheetrefs" "${INTERSHEET_REFS}" (at 22.7061 58.42 0)
-      (effects (font (size 1.27 1.27)) (justify right) hide)
-    )
-  )
-  (global_label "SEL2_MotorR" (shape input) (at 170.815 74.93 180) (fields_autoplaced)
-    (effects (font (size 1.27 1.27)) (justify right))
-    (property "Intersheetrefs" "${INTERSHEET_REFS}" (at 155.8142 74.93 0)
-      (effects (font (size 1.27 1.27)) (justify right) hide)
-    )
-  )
-  (global_label "SEL1_MotorR" (shape input) (at 170.815 58.42 180) (fields_autoplaced)
-    (effects (font (size 1.27 1.27)) (justify right))
-    (property "Intersheetrefs" "${INTERSHEET_REFS}" (at 155.8142 58.42 0)
-      (effects (font (size 1.27 1.27)) (justify right) hide)
-    )
+  (hierarchical_label "PWM_MotorR" (shape input) (at 170.815 66.675 180) (fields_autoplaced)
+    (effects (font (size 1.27 1.27) bold) (justify right))
+  )
+  (hierarchical_label "SEL1_MotorL" (shape input) (at 37.465 58.42 180) (fields_autoplaced)
+    (effects (font (size 1.27 1.27) bold) (justify right))
+  )
+  (hierarchical_label "SEL2_MotorL" (shape input) (at 37.465 74.93 180) (fields_autoplaced)
+    (effects (font (size 1.27 1.27) bold) (justify right))
+  )
+  (hierarchical_label "SEL2_MotorR" (shape input) (at 170.815 74.93 180) (fields_autoplaced)
+    (effects (font (size 1.27 1.27) bold) (justify right))
+  )
+  (hierarchical_label "PWM_MotorL" (shape input) (at 37.465 66.675 180) (fields_autoplaced)
+    (effects (font (size 1.27 1.27) bold) (justify right))
+  )
+  (hierarchical_label "SEL1_MotorR" (shape input) (at 170.815 58.42 180) (fields_autoplaced)
+    (effects (font (size 1.27 1.27) bold) (justify right))
   )
   (symbol (lib_id "Device:R") (at 50.8 85.725 0) (unit 1)
